File: hardware/droneSTM32/peripherals.kicad_sch (KiCad schematic)
At the start: 0 parts

Commit message: commit mpu6050 update
Parts:
- added C401, C403: 100nF, symbol Device:C_Small
- added C402: 2.2nF, symbol Device:C_Small
- added C404: 10nF, symbol Device:C_Small
- added R401, R402, R403: 4.7k, Sensor_Motion:InvenSense_QFN-24_4x4mm_P0.5mm, symbol Device:R_Small
- added U401: MPU-6050, Sensor_Motion:InvenSense_QFN-24_4x4mm_P0.5mm, symbol Sensor_Motion:MPU-6050
Connections:
- new net: C403.1, U401.10 (REGOUT)
- new net: C402.1, U401.20 (CPOUT)
- new net: R401.1, U401.9 (AD0)
- new net +3.3V: C401.1, C404.1, R402.1, R403.1, U401.13 (VDD), U401.8 (VLOGIC)
- new net GND: C401.2, C402.2, C403.2, C404.2, R401.2, U401.1 (CLKIN), U401.11 (FSYNC), U401.18 (GND)
- new net I2C2_SCL: R403.2, U401.23 (SCL)
- new net I2C2_SDA: R402.2, U401.24 (SDA)
- no-connect marks 0 -> 3
